Commit message: Clean up code and made changes to workflow.

File: ekg_auv_testing/urdf/basic_beacon.xacro (robot description, xacro)
@@ -6,5 +6,5 @@
     <xacro:include filename="$(find uuv_gazebo_ros_plugins)/urdf/snippets.xacro"/>
     <!-- Properties -->
-    <xacro:property name="mass" value="0.85"/>
+    <xacro:property name="mass" value="0.45"/>
     <xacro:property name="radius" value="0.05"/>
     <xacro:property name="length" value="0.3"/>
@@ -30,9 +30,9 @@
             <inertial>
                 <mass value="${mass}"/>
-                <origin xyz="0 1 0" rpy="0 0 0"/>
+                <!--origin xyz="0 1 0" rpy="0 0 0"/-->
                 <inertia
                     ixx="0.12" ixy="0.0" ixz="0.0"
                     iyy="0.12" iyz="0.0"
-                    izz="0.11"/>
+                    izz="0.106"/>
             </inertial>
         </link>
@@ -64,4 +64,11 @@
                 <sigma>0.0</sigma>
             </plugin>
+            <!--plugin name="beacon_controller" filename="libSimple3dMovePlugin.so">
+                <commandTopic>cmd_vel</commandTopic>
+                <odometryTopic>odom</odometryTopic>
+                <odometryFrame>odom</odometryFrame>
+                <odometryRate>20.0</odometryRate>
+                <robotBaseFrame>base_footprint</robotBaseFrame>
+            </plugin-->
         </gazebo>
     </xacro:macro>

Commit message: Simple deadreckoning graphing

File: ekg_auv_testing/urdf/basic_beacon.xacro (robot description, xacro)
@@ -64,12 +64,26 @@
                 <sigma>0.0</sigma>
             </plugin>
-            <!--plugin name="beacon_controller" filename="libSimple3dMovePlugin.so">
-                <commandTopic>cmd_vel</commandTopic>
-                <odometryTopic>odom</odometryTopic>
-                <odometryFrame>odom</odometryFrame>
-                <odometryRate>20.0</odometryRate>
-                <robotBaseFrame>base_footprint</robotBaseFrame>
-            </plugin-->
         </gazebo>
+        <!-- Pressure Sensor -->
+        <xacro:pressure_plugin_macro
+            namespace="${namespace}"
+            suffix=""
+            parent_link="${namespace}/base_link"
+            topic="pressure"
+            mass="0.015"
+            update_rate="10"
+            range="1362"
+            noise_sigma="3.0"
+            noise_amplitude="0.0"
+            estimateDepth="true"
+            standardPressure="101.325"
+            kPaPerM="9.80638">
+            <inertia ixx="0.00001" ixy="0.0" ixz="0.0" iyy="0.00001" iyz="0.0" izz="0.00001" />
+            <origin xyz="0.0 0.0 0.0" rpy="0 ${0.355556*pi} 0" />
+        </xacro:pressure_plugin_macro>
+        <!-- IMU Sensor -->
+        <xacro:include filename="$(find glider_hybrid_whoi_description)/urdf/uw_hector_imu_plugin.xacro"/>
+        <!-- GPS Sensor -->
+        <!--xacro:include filename="$(find glider_hybrid_whoi_description)/urdf/uw_hector_gps_plugin.xacro"/-->
     </xacro:macro>
 </robot>

Commit message: Created Plugin functionality in Python and made changes to Gazebo plugin

File: ekg_auv_testing/urdf/basic_beacon.xacro (robot description, xacro)
@@ -9,7 +9,9 @@
     <xacro:property name="radius" value="0.05"/>
     <xacro:property name="length" value="0.3"/>
-    <xacro:property name="namespace" value="basic_beacon"/>
+    <xacro:property name="namespace" default="basic_beacon"/>
+    <xacro:property name="transceiver_id" default="168"/>
+    <xacro:property name="transponder_id" default="1"/>
     <!-- Robot Definition -->
-    <xacro:macro name="basic_beacon" params="namespace debug inertial_reference_frame">
+    <xacro:macro name="basic_beacon" params="namespace debug transceiver_id transponder_id inertial_reference_frame">
         <link name="${namespace}/base_link">
             <visual name="visual">
@@ -28,12 +30,12 @@
                 </geometry>
             </collision>
-            <inertial>
+            <!--inertial>
                 <mass value="${mass}"/>
-                <!--origin xyz="0 1 0" rpy="0 0 0"/-->
+                <origin xyz="0 1 0" rpy="0 0 0"/>
                 <inertia
                     ixx="0.12" ixy="0.0" ixz="0.0"
                     iyy="0.12" iyz="0.0"
                     izz="0.106"/>
-            </inertial>
+            </inertial-->
         </link>
         <gazebo reference="link">
@@ -42,25 +44,23 @@
         <!-- Set up USBL Plugin for TX and RX -->
         <gazebo>
-            <plugin name="${namespace}_tx" filename="libtransceiverPlugin.so">
-                <namespace>USBL_Transciever</namespace>
-                <transponder_device>trasnponder_manufacturer</transponder_device>
-                <transponder_ID>1</transponder_ID>
-                <transceiver_device>tranceiver_manufacturer</transceiver_device>
-                <transceiver_ID>168</transceiver_ID>
-                <enable_ping_scheduler>0</enable_ping_scheduler>
-                <transponder_attached_object>sphere</transponder_attached_object>
+            <!--plugin name="${namespace}_tx" filename="libtransceiverPlugin.so">
+                <namespace>USBL</namespace>
+                <transponder_device>transponder_manufacturer</transponder_device>
+                <transponder_ID>${transponder_id}</transponder_ID>
+                <transceiver_device>transceiver_manufacturer</transceiver_device>
+                <transceiver_ID>${transceiver_id}</transceiver_ID>
+                <enable_ping_scheduler>false</enable_ping_scheduler>
+                <transponder_attached_object>${namespace}</transponder_attached_object>
                 <interrogation_mode>common</interrogation_mode>
                 <sound_speed>1540.0</sound_speed>
                 <ping_freq>2</ping_freq>
-            </plugin>
-            <plugin name='${namespace}_rx' filename='libtransponderPlugin.so'>
-                <namespace>USBL_Transponder</namespace>
-                <transponder_device>trasnponder_manufacturer</transponder_device>
-                <transponder_ID>1</transponder_ID>
-                <transceiver_device>tranceiver_manufacturer</transceiver_device>
-                <transceiver_ID>168</transceiver_ID>
-                <sound_speed>1540.0</sound_speed>
-                <mu>0</mu>
-                <sigma>0.0</sigma>
+            </plugin-->
+            <plugin name="${namespace}_control" filename="libekg_spatial_move.so">
+                <robotNamespace>${namespace}</robotNamespace>
+                <commandTopic>cmd_vel</commandTopic>
+                <odometryTopic>${namespace}/pose_gt</odometryTopic>
+                <odometryFrame>odom</odometryFrame>
+                <robotBaseFrame>base_footprint</robotBaseFrame>
+                <odometryRate>20.0</odometryRate>
             </plugin>
         </gazebo>

File: ekg_auv_testing/urdf/basic_beacon_default.urdf.xacro (robot description, xacro)
@@ -3,4 +3,6 @@
   <xacro:arg name="debug" default="0"/>
   <xacro:arg name="namespace" default="basic_beacon"/>
+  <xacro:arg name="transceiver_id" default="168"/>
+  <xacro:arg name="transponder_id" default="1"/>
   <xacro:arg name="inertial_reference_frame" default="world"/>
   <!-- Include beacon macro file -->
@@ -10,4 +12,6 @@
     namespace="$(arg namespace)"
     debug="$(arg debug)"
+    transceiver_id= "$(arg transceiver_id)"
+    transponder_id="$(arg transponder_id)"
     inertial_reference_frame="$(arg inertial_reference_frame)"/>
   <!-- Joint state publisher plugin -->
